File: hardware/KiCad/FPGA v1.0.kicad_sch (KiCad schematic)
At the start: 4 parts

Commit message: Add files via upload
v1.1
Other:
- note added: "V1.1 designed by Cris R. Martinez Hernandez"
- note added: "Vision Core v1.1"
- note removed: "Draft 1.0 prepared by Cris R. Martinez Hernandez"
- note removed: "Vision Core v1.0"
